File: preamp.brd (EAGLE design)
At the start: 100 x 92.7 mm, 73 parts, among them IC1 INA217DW, IC2 OPA134U, IC3 PCM1808, IC4 12.288MHz, IC5 REG1117

Commit message: comment after soldering
Parts:
- added R16: 0, rcl:R0805
- C22, C29, C31: value 47 -> 100u
- L1, L2: value (none) -> 100u
- R5: value (none) -> G
Connections:
- removed net N$15: C19.2, IC2.3, R11.2, R13.1
- new net N$29: C19.2, IC2.3, R11.2, R13.1, R16.2, R3.1, R4.1
- net AGND: now also R16.1; no longer R3.1, R4.1
Routing:
- net N$15: track 9.98 -> 0.00 mm
- net AGND: track 133.0 -> 129.8 mm
Changed lines of the file:
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@@
 <element name="R3" library="rcl" package="R0805" value="2.2k" x="23.495" y="31.115" rot="R270"/>
 <element name="R4" library="rcl" package="R0805" value="2.2k" x="23.495" y="36.195" rot="R90"/>
-<element name="R5" library="rcl" package="R0805" value="" x="42.545" y="44.45" rot="R180"/>
+<element name="R5" library="rcl" package="R0805" value="G" x="42.545" y="44.45" rot="R180"/>
 <element name="R6" library="rcl" package="R0805" value="1M" x="55.245" y="36.83" rot="R180"/>
 <element name="J3" library="con-amp" package="10X02MTA" value="" x="24.765" y="44.45"/>
@@
 <element name="C20" library="rcl" package="C0805" value="0.1" x="64.77" y="14.605"/>
 <element name="C21" library="rcl" package="C0805" value="0.1" x="53.34" y="15.875" rot="R90"/>
-<element name="C22" library="rcl" package="153CLV-0605" value="47" x="48.895" y="18.415" rot="R270"/>
+<element name="C22" library="rcl" package="153CLV-0605" value="100u" x="48.895" y="18.415" rot="R270"/>
 <element name="C23" library="rcl" package="C0805" value="0.1" x="24.765" y="4.445" rot="R270"/>
 <element name="C24" library="rcl" package="C0805" value="0.1" x="31.115" y="7.62" rot="R90"/>
@@
 <element name="J8" library="con-amp" package="10X04MTA" value="" x="9.525" y="11.43" rot="R270"/>
 <element name="J9" library="con-amp" package="10X02MTA" value="" x="64.135" y="20.32" rot="R90"/>
-<element name="L1" library="rcl" package="L3225M" value="" x="43.815" y="6.985" rot="R90"/>
-<element name="L2" library="rcl" package="L3225M" value="" x="53.975" y="6.985" rot="R270"/>
-<element name="C29" library="rcl" package="153CLV-0605" value="47" x="48.895" y="5.715" rot="R90"/>
+<element name="L1" library="rcl" package="L3225M" value="100u" x="43.815" y="6.985" rot="R90"/>
+<element name="L2" library="rcl" package="L3225M" value="100u" x="53.975" y="6.985" rot="R270"/>
+<element name="C29" library="rcl" package="153CLV-0605" value="100u" x="48.895" y="5.715" rot="R90"/>
 <element name="C30" library="rcl" package="153CLV-0605" value="47" x="63.5" y="5.715" rot="R90"/>
-<element name="C31" library="rcl" package="153CLV-0605" value="47" x="38.735" y="5.715" rot="R90"/>
+<element name="C31" library="rcl" package="153CLV-0605" value="100u" x="38.735" y="5.715" rot="R90"/>
 <element name="R17" library="rcl" package="R0805" value="0" x="57.785" y="2.54"/>
 <element name="R13" library="rcl" package="R0805" value="0" x="62.23" y="27.94"/>
@@
 <element name="C32" library="rcl" package="153CLV-0605" value="47" x="57.15" y="66.675" rot="R90"/>
 <element name="C33" library="rcl" package="153CLV-0605" value="47" x="57.15" y="56.515" rot="R90"/>
+<element name="R16" library="rcl" package="R0805" value="0" x="-14.605" y="-15.875"/>
 </elements>
 <signals>
@@
 <signal name="AGND">
 <contactref element="C3" pad="1"/>
-<contactref element="R3" pad="1"/>
-<contactref element="R4" pad="1"/>
 <contactref element="C2" pad="1"/>
 <contactref element="J2" pad="2"/>
@@
 <wire x1="53.975" y1="40.64" x2="55.565" y2="40.64" width="0.6096" layer="1"/>
 <wire x1="13.335" y1="33.655" x2="23.495" y2="33.655" width="0.6096" layer="1"/>
-<wire x1="23.495" y1="33.655" x2="23.495" y2="32.065" width="0.6096" layer="1"/>
-<wire x1="23.495" y1="35.245" x2="23.495" y2="33.655" width="0.6096" layer="1"/>
 <wire x1="10.16" y1="34.925" x2="12.065" y2="34.925" width="0.6096" layer="1"/>
 <wire x1="12.065" y1="34.925" x2="13.335" y2="33.655" width="0.6096" layer="1"/>
@@
 <wire x1="34.925" y1="71.755" x2="30.16" y2="71.755" width="0.6096" layer="1"/>
 <wire x1="30.16" y1="71.755" x2="28.89" y2="70.485" width="0.6096" layer="1"/>
+<contactref element="R16" pad="1"/>
 <wire x1="26.035" y1="44.45" x2="26.99" y2="53.34" width="0" layer="19" extent="1-1"/>
+<wire x1="-15.555" y1="-15.875" x2="10.16" y2="34.925" width="0" layer="19" extent="1-1"/>
 </signal>
 <signal name="V+">
@@
 <wire x1="29.21" y1="55.88" x2="29.21" y2="53.66" width="0.6096" layer="1"/>
 <wire x1="29.21" y1="53.66" x2="28.89" y2="53.34" width="0.6096" layer="1"/>
-</signal>
-<signal name="N$15">
-<contactref element="IC2" pad="3"/>
-<contactref element="R11" pad="2"/>
-<contactref element="C19" pad="2"/>
-<wire x1="60.96" y1="33.02" x2="57.8612" y2="33.02" width="0.6096" layer="1"/>
-<contactref element="R13" pad="1"/>
-<wire x1="61.28" y1="27.94" x2="61.28" y2="28.255" width="0.6096" layer="1"/>
-<wire x1="61.28" y1="28.255" x2="60.96" y2="28.575" width="0.254" layer="1"/>
-<wire x1="60.96" y1="28.575" x2="60.96" y2="30.795" width="0.6096" layer="1"/>
-<wire x1="60.96" y1="30.795" x2="61.28" y2="31.115" width="0.254" layer="1"/>
-<wire x1="61.28" y1="31.115" x2="61.28" y2="31.43" width="0.254" layer="1"/>
-<wire x1="61.28" y1="31.43" x2="60.96" y2="31.75" width="0.6096" layer="1"/>
-<wire x1="60.96" y1="31.75" x2="60.96" y2="33.02" width="0.6096" layer="1"/>
-<wire x1="60.96" y1="33.02" x2="60.96" y2="33.97" width="0.6096" layer="1"/>
-<wire x1="60.96" y1="33.97" x2="61.28" y2="34.29" width="0.6096" layer="1"/>
 </signal>
 <signal name="N$8">
@@
 <wire x1="66.04" y1="36.83" x2="65.405" y2="37.465" width="0.6096" layer="1"/>
 </signal>
+<signal name="N$29">
+<contactref element="R3" pad="1"/>
+<contactref element="R4" pad="1"/>
+<contactref element="R16" pad="2"/>
+<contactref element="C19" pad="2"/>
+<contactref element="R11" pad="2"/>
+<contactref element="IC2" pad="3"/>
+<contactref element="R13" pad="1"/>
+<wire x1="61.28" y1="31.115" x2="61.28" y2="34.29" width="0" layer="19" extent="1-1"/>
+<wire x1="61.28" y1="27.94" x2="61.28" y2="31.115" width="0" layer="19" extent="1-1"/>
+<wire x1="57.8612" y1="33.02" x2="61.28" y2="34.29" width="0" layer="19" extent="1-1"/>
+<wire x1="23.495" y1="32.065" x2="57.8612" y2="33.02" width="0" layer="19" extent="1-1"/>
+<wire x1="23.495" y1="35.245" x2="23.495" y2="32.065" width="0" layer="19" extent="1-1"/>
+<wire x1="-13.655" y1="-15.875" x2="23.495" y2="32.065" width="0" layer="19" extent="1-1"/>
+</signal>
 </signals>
