File: preamp.sch (EAGLE design)
At the start: 73 parts, among them IC1 INA217DW, IC2 OPA134U, IC3 PCM1808, IC4 12.288MHz, IC5 REG1117

Commit message: comment after soldering
Parts:
- added R16: 0, rcl:R-EU_R0805
- C22, C29, C31: value 47 -> 100u
- L1, L2: value (none) -> 100u
- R5: value (none) -> G
Connections:
- removed net N$15: C19.2, IC2.+IN, R11.2, R13.1
- new net N$29: C19.2, IC2.+IN, R11.2, R13.1, R16.2, R3.1, R4.1
- net AGND: now also R16.1; no longer R3.1, R4.1
Other:
- note added: "G = 1 + 10000/Rg"
- note added: "G = 104 Rg = 97"
- note added: "G = 74 Rg = 137"
- note added: "С2 и С3 перенести ближе к ИС"
- note added: "на выход REF поставить делитель после повторитель как в дипломе opa184 не нужен, с повторителя сразу на ИС"
- note added: "на плате сделать просто дорожку"
- note removed: "1) нагрузочные резисторы для источника, потом выпаюются 2) источники подключить через нульовые резисторы, тоже для проверки 3) по пути от источника поставить smd штыри, пусть будут площадки для проверки 4) резистор отвечающий за усиление, оставить ему место на разводке чтобы можно было подбирать 5) усилители сделать с возможностью отеделения, блок питания так же"
Changed lines of the file:
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@@
 <part name="R3" library="rcl" deviceset="R-EU_" device="R0805" value="2.2k"/>
 <part name="R4" library="rcl" deviceset="R-EU_" device="R0805" value="2.2k"/>
-<part name="R5" library="rcl" deviceset="R-EU_" device="R0805"/>
+<part name="R5" library="rcl" deviceset="R-EU_" device="R0805" value="G"/>
 <part name="R6" library="rcl" deviceset="R-EU_" device="R0805" value="1M"/>
 <part name="C1" library="rcl" deviceset="C-EU" device="C0805" value="0.1"/>
@@
 <part name="GND4" library="supply1" deviceset="GND" device=""/>
 <part name="GND5" library="supply1" deviceset="GND" device=""/>
-<part name="C22" library="rcl" deviceset="CPOL-EU" device="153CLV-0605" value="47"/>
+<part name="C22" library="rcl" deviceset="CPOL-EU" device="153CLV-0605" value="100u"/>
 <part name="C23" library="rcl" deviceset="C-EU" device="C0805" value="0.1"/>
 <part name="C24" library="rcl" deviceset="C-EU" device="C0805" value="0.1"/>
@@
 <part name="+3V2" library="supply1" deviceset="+3V3" device=""/>
 <part name="+3V3" library="supply1" deviceset="+3V3" device=""/>
-<part name="L1" library="rcl" deviceset="L-US" device="L3225M"/>
-<part name="L2" library="rcl" deviceset="L-US" device="L3225M"/>
-<part name="C29" library="rcl" deviceset="CPOL-EU" device="153CLV-0605" value="47"/>
+<part name="L1" library="rcl" deviceset="L-US" device="L3225M" value="100u"/>
+<part name="L2" library="rcl" deviceset="L-US" device="L3225M" value="100u"/>
+<part name="C29" library="rcl" deviceset="CPOL-EU" device="153CLV-0605" value="100u"/>
 <part name="P+10" library="supply1" deviceset="VCC" device=""/>
 <part name="C30" library="rcl" deviceset="CPOL-EU" device="153CLV-0605" value="47"/>
-<part name="C31" library="rcl" deviceset="CPOL-EU" device="153CLV-0605" value="47"/>
+<part name="C31" library="rcl" deviceset="CPOL-EU" device="153CLV-0605" value="100u"/>
 <part name="R17" library="rcl" deviceset="R-EU_" device="R0805" value="0"/>
 <part name="R13" library="rcl" deviceset="R-EU_" device="R0805" value="0"/>
@@
 <part name="C32" library="rcl" deviceset="CPOL-EU" device="153CLV-0605" value="47"/>
 <part name="C33" library="rcl" deviceset="CPOL-EU" device="153CLV-0605" value="47"/>
+<part name="R16" library="rcl" deviceset="R-EU_" device="R0805" value="0"/>
 </parts>
 <sheets>
 <sheet>
 <plain>
-<text x="165.1" y="269.24" size="2.54" layer="91">1) нагрузочные резисторы для источника, потом выпаюются
-2) источники подключить через нульовые резисторы, тоже для проверки
-3) по пути от источника поставить smd штыри, пусть будут площадки для проверки
-4) резистор отвечающий за усиление, оставить ему место на разводке чтобы можно было подбирать
-5) усилители сделать с возможностью отеделения, блок питания так же</text>
 <text x="-30.48" y="81.28" size="1.778" layer="91">GND</text>
 <text x="-30.48" y="83.82" size="1.778" layer="91">INL</text>
@@
 <text x="-30.48" y="195.58" size="1.778" layer="91">GND</text>
 <text x="-30.48" y="198.12" size="1.778" layer="91">5V</text>
+<text x="175.26" y="50.8" size="1.778" layer="91">на выход REF поставить делитель после повторитель как в дипломе
+opa184 не нужен, с повторителя сразу на ИС</text>
+<text x="111.76" y="99.06" size="1.778" layer="91">С2 и С3 перенести ближе к ИС</text>
+<text x="53.34" y="101.6" size="1.778" layer="91">G = 1 + 10000/Rg</text>
+<text x="50.8" y="109.22" size="1.778" layer="91">G = 74
+Rg = 137</text>
+<text x="68.58" y="109.22" size="1.778" layer="91">G = 104
+Rg = 97</text>
+<text x="353.06" y="55.88" size="1.778" layer="91">на плате сделать просто дорожку</text>
 </plain>
 <instances>
@@
 <instance part="AGND2" gate="VR1" x="96.52" y="38.1"/>
 <instance part="AGND3" gate="VR1" x="96.52" y="96.52"/>
-<instance part="AGND4" gate="VR1" x="50.8" y="30.48"/>
+<instance part="AGND4" gate="VR1" x="50.8" y="10.16"/>
 <instance part="P+4" gate="1" x="106.68" y="121.92"/>
 <instance part="P+5" gate="1" x="40.64" y="114.3"/>
@@
 <instance part="C32" gate="G$1" x="99.06" y="195.58"/>
 <instance part="C33" gate="G$1" x="99.06" y="177.8"/>
+<instance part="R16" gate="G$1" x="50.8" y="20.32" rot="R90"/>
 </instances>
 <busses>
@@
 <pinref part="AGND2" gate="VR1" pin="AGND"/>
 <wire x1="96.52" y1="43.18" x2="96.52" y2="40.64" width="0.1524" layer="91"/>
-</segment>
-<segment>
-<pinref part="R3" gate="G$1" pin="1"/>
-<pinref part="AGND4" gate="VR1" pin="AGND"/>
-<wire x1="50.8" y1="40.64" x2="50.8" y2="38.1" width="0.1524" layer="91"/>
-<pinref part="R4" gate="G$1" pin="1"/>
-<wire x1="50.8" y1="38.1" x2="50.8" y2="33.02" width="0.1524" layer="91"/>
-<wire x1="50.8" y1="38.1" x2="55.88" y2="38.1" width="0.1524" layer="91"/>
-<wire x1="55.88" y1="38.1" x2="55.88" y2="40.64" width="0.1524" layer="91"/>
-<junction x="50.8" y="38.1"/>
 </segment>
 <segment>
@@
 <wire x1="147.32" y1="78.74" x2="147.32" y2="71.12" width="0.1524" layer="91"/>
 </segment>
+<segment>
+<pinref part="AGND4" gate="VR1" pin="AGND"/>
+<pinref part="R16" gate="G$1" pin="1"/>
+<wire x1="50.8" y1="12.7" x2="50.8" y2="15.24" width="0.1524" layer="91"/>
+</segment>
 </net>
 <net name="V+" class="0">
@@
 <wire x1="45.72" y1="170.18" x2="45.72" y2="167.64" width="0.1524" layer="91"/>
 <junction x="45.72" y="167.64"/>
-</segment>
-</net>
-<net name="N$15" class="0">
-<segment>
-<pinref part="IC2" gate="G$1" pin="+IN"/>
-<wire x1="137.16" y1="43.18" x2="139.7" y2="43.18" width="0.1524" layer="91"/>
-<pinref part="R11" gate="G$1" pin="2"/>
-<wire x1="139.7" y1="38.1" x2="139.7" y2="43.18" width="0.1524" layer="91"/>
-<pinref part="C19" gate="G$1" pin="2"/>
-<wire x1="139.7" y1="43.18" x2="147.32" y2="43.18" width="0.1524" layer="91"/>
-<wire x1="147.32" y1="43.18" x2="147.32" y2="38.1" width="0.1524" layer="91"/>
-<junction x="139.7" y="43.18"/>
-<wire x1="152.4" y1="43.18" x2="147.32" y2="43.18" width="0.1524" layer="91"/>
-<junction x="147.32" y="43.18"/>
-<pinref part="R13" gate="G$1" pin="1"/>
-<wire x1="152.4" y1="43.18" x2="152.4" y2="48.26" width="0.1524" layer="91"/>
 </segment>
 </net>
@@
 </segment>
 </net>
+<net name="N$29" class="0">
+<segment>
+<pinref part="R3" gate="G$1" pin="1"/>
+<wire x1="50.8" y1="40.64" x2="50.8" y2="38.1" width="0.1524" layer="91"/>
+<pinref part="R4" gate="G$1" pin="1"/>
+<wire x1="50.8" y1="38.1" x2="55.88" y2="38.1" width="0.1524" layer="91"/>
+<wire x1="55.88" y1="38.1" x2="55.88" y2="40.64" width="0.1524" layer="91"/>
+<pinref part="R16" gate="G$1" pin="2"/>
+<wire x1="50.8" y1="25.4" x2="50.8" y2="30.48" width="0.1524" layer="91"/>
+<junction x="50.8" y="38.1"/>
+<wire x1="50.8" y1="30.48" x2="50.8" y2="38.1" width="0.1524" layer="91"/>
+<wire x1="50.8" y1="30.48" x2="116.84" y2="30.48" width="0.1524" layer="91"/>
+<wire x1="116.84" y1="30.48" x2="116.84" y2="10.16" width="0.1524" layer="91"/>
+<pinref part="IC2" gate="G$1" pin="+IN"/>
+<wire x1="137.16" y1="43.18" x2="139.7" y2="43.18" width="0.1524" layer="91"/>
+<pinref part="R11" gate="G$1" pin="2"/>
+<wire x1="139.7" y1="38.1" x2="139.7" y2="43.18" width="0.1524" layer="91"/>
+<pinref part="C19" gate="G$1" pin="2"/>
+<wire x1="139.7" y1="43.18" x2="147.32" y2="43.18" width="0.1524" layer="91"/>
+<wire x1="147.32" y1="43.18" x2="147.32" y2="38.1" width="0.1524" layer="91"/>
+<junction x="139.7" y="43.18"/>
+<wire x1="152.4" y1="43.18" x2="147.32" y2="43.18" width="0.1524" layer="91"/>
+<junction x="147.32" y="43.18"/>
+<pinref part="R13" gate="G$1" pin="1"/>
+<wire x1="152.4" y1="43.18" x2="152.4" y2="48.26" width="0.1524" layer="91"/>
+<wire x1="116.84" y1="10.16" x2="152.4" y2="10.16" width="0.1524" layer="91"/>
+<wire x1="152.4" y1="10.16" x2="152.4" y2="43.18" width="0.1524" layer="91"/>
+<junction x="50.8" y="30.48"/>
+<junction x="152.4" y="43.18"/>
+</segment>
+</net>
